File: Mini/V3.0/V3.0.kicad_sch (KiCad schematic)
At the start: 23 parts, among them J1 UJC-HP2-3-SMT-TR, J2 Eurorack_Power_16pin_Shrouded, J3 Eurorack_Power_16pin_Shrouded, J6 VN02A1500000G

Commit message: Adding PDF schematic
Parts:
- D2, D3, D4, J2, J3, J6, PS1: now fitted
