File: EuroPlatvorm/EuroPlatvorm.kicad_sch (KiCad schematic)
At the start: 0 parts

Commit message: Add ESP32-C6 core + dual-source power schematic with carrier headers
- Power: Doepfer +12V (F1 PTC, D1 SS34 -> TPS54202 buck @ 3.43V,
  R1/R2 100k/21k) and USB-C VBUS (F2 PTC -> AMS1117-3.3); buck
  dominates when both sources attached
- Firmware via native ESP32-C6 USB-Serial/JTAG (IO12/13) with
  USBLC6-2SC6 ESD - CH340C intentionally dropped
- Strapping per datasheet: EN 10k+1uF + RST button, IO9 10k PU +
  BOOT button, IO8 10k PU, IO15 float
- J3/J4 1x14 carrier headers: all 23 GPIOs + +12V/-12V/+3V3/GND,
  netlabel-routed for free placement during layout
- Verified: kicad-cli ERC 0/0, netlist connectivity asserted,
  analyzer triaged (PP-001 false positive, EN float by design)
- Reference docs: TPS54202/CH340C datasheets, ESP32-C6-WROOM-1
  datasheet extraction
Parts:
- added C1: 10uF 25V, Capacitor_SMD:C_1206_3216Metric, symbol platvorm:C
- added C10, C4, C5, C8: 22uF 10V, Capacitor_SMD:C_0805_2012Metric, symbol platvorm:C
- added C11, C2, C3: 100nF, Capacitor_SMD:C_0603_1608Metric, symbol platvorm:C
- added C6: 56pF, Capacitor_SMD:C_0603_1608Metric, symbol platvorm:C
- added C7: 10uF 10V, Capacitor_SMD:C_0805_2012Metric, symbol platvorm:C
- added C9: 1uF, Capacitor_SMD:C_0603_1608Metric, symbol platvorm:C
- added D1: SS34, Diode_SMD:D_SMA, symbol platvorm:D_Schottky
- added D2: LED_Green, LED_SMD:LED_0603_1608Metric, symbol platvorm:LED
- added F1, F2: 500mA PTC, Fuse:Fuse_1206_3216Metric, symbol platvorm:Polyfuse
- added J1: Eurorack_Power_2x5, Connector_IDC:IDC-Header_2x05_P2.54mm_Vertical, symbol platvorm:Conn_02x05_Odd_Even
- added J2: USB_C_Receptacle_USB2.0, platvorm_custom:USB-C_SMD-TYPE-C-31-M-12_1, symbol platvorm:USB_C_Receptacle_USB2.0_16P
- added J3, J4: Conn_01x14, Connector_PinHeader_2.54mm:PinHeader_1x14_P2.54mm_Vertical, symbol platvorm:Conn_01x14
- added L1: 10uH, platvorm_custom:IND-SMD_L6.0-W6.0, symbol platvorm:L
- added R1: 100k, Resistor_SMD:R_0603_1608Metric, symbol platvorm:R
- added R2: 21k, Resistor_SMD:R_0603_1608Metric, symbol platvorm:R
- added R3, R4: 5.1k, Resistor_SMD:R_0603_1608Metric, symbol platvorm:R
- added R5, R6, R7: 10k, Resistor_SMD:R_0603_1608Metric, symbol platvorm:R
- added R8: 1k, Resistor_SMD:R_0603_1608Metric, symbol platvorm:R
- added SW1: RST, platvorm_custom:SW_TS-1187A, symbol platvorm:SW_Push
- added SW2: BOOT, platvorm_custom:SW_TS-1187A, symbol platvorm:SW_Push
- added U1: TPS54202DDCR, Package_TO_SOT_SMD:SOT-23-6, symbol platvorm:TPS54202
- added U2: AMS1117-3.3, Package_TO_SOT_SMD:SOT-223-3_TabPin2, symbol platvorm:AMS1117-3.3
- added U3: USBLC6-2SC6, Package_TO_SOT_SMD:SOT-23-6, symbol platvorm:USBLC6-2SC6
- added U4: ESP32-C6-WROOM-1-N4, PCM_Espressif:ESP32-C6-WROOM-1, symbol PCM_Espressif:ESP32-C6-WROOM-1
Connections:
- new net: C3.1, L1.1, U1.2 (SW)
- new net: C1.1, C2.1, D1.1 (K), U1.3 (VIN)
- new net: C6.2, R1.2, R2.1, U1.4 (FB)
- new net: C3.2, U1.6 (BOOT)
- new net: D1.2 (A), F1.2
- new net: C9.1, R5.2, SW1.2, U4.3 (EN/CHIP_PU)
- new net: D2.2 (A), R8.2
- new net: J2.A5 (CC1), R3.1
- new net: F2.2, J2.A4B9 (VBUS), J2.B4A9 (VBUS)
- new net: J2.B5 (CC2), R4.1
- new net +12V: F1.1, J1.10 (Pin_10), J1.9 (Pin_9), J3.2 (Pin_2)
- new net +3V3: C10.2, C11.2, C4.1, C5.1, C6.1, C8.1, J3.1 (Pin_1), L1.2, R1.1, R5.1, R6.1, R7.1, R8.1, U2.2 (VO), U4.2 (3V3)
- new net -12V: J1.1 (Pin_1), J1.2 (Pin_2), J3.3 (Pin_3)
- new net GND: C1.2, C10.1, C11.1, C2.2, C4.2, C5.2, C7.2, C8.2, C9.2, D2.1 (K), J1.3 (Pin_3), J1.4 (Pin_4), J1.5 (Pin_5), J1.6 (Pin_6), J1.7 (Pin_7), J1.8 (Pin_8), J2.1 (SHIELD), J2.2 (SHIELD), J2.3 (SHIELD), J2.4 (SHIELD), J2.A1B12 (GND), J2.B1A12 (GND), J3.14 (Pin_14), J4.14 (Pin_14), R2.2, R3.2, R4.2, SW1.1, SW2.2, U1.1 (GND), U2.1 (GND), U3.2 (GND), U4.1 (GND), U4.28 (GND), U4.29 (GND)
- new net GPIO0: J3.4 (Pin_4), U4.8 (GPIO0/ADC1_CH0/XTAL_32K_P)
- new net GPIO1: J3.5 (Pin_5), U4.9 (GPIO1/ADC1_CH1/XTAL_32K_N)
- new net GPIO10: J3.12 (Pin_12), U4.11 (GPIO10)
- new net GPIO11: J4.11 (Pin_11), U4.12 (GPIO11)
- new net GPIO15: J3.13 (Pin_13), U4.23 (GPIO15)
- new net GPIO16: J4.7 (Pin_7), U4.25 (U0TXD/GPIO16)
- new net GPIO17: J4.8 (Pin_8), U4.24 (U0RXD/GPIO17)
- new net GPIO18: J4.1 (Pin_1), U4.16 (GPIO18)
- new net GPIO19: J4.2 (Pin_2), U4.17 (GPIO19)
- new net GPIO2: J3.6 (Pin_6), U4.27 (GPIO2/ADC1_CH2)
- new net GPIO20: J4.3 (Pin_3), U4.18 (GPIO20)
- new net GPIO21: J4.4 (Pin_4), U4.19 (GPIO21)
- new net GPIO22: J4.5 (Pin_5), U4.20 (GPIO22)
- new net GPIO23: J4.6 (Pin_6), U4.21 (GPIO23)
- new net GPIO3: J3.7 (Pin_7), U4.26 (GPIO3/ADC1_CH3)
- new net GPIO4: J3.8 (Pin_8), U4.4 (MTMS/GPIO4/ADC1_CH4)
- new net GPIO5: J3.9 (Pin_9), U4.5 (MTDI/GPIO5/ADC1_CH5)
- new net GPIO6: J3.10 (Pin_10), U4.6 (MTCK/GPIO6/ADC1_CH6)
- new net GPIO7: J3.11 (Pin_11), U4.7 (MTDO/GPIO7)
- new net GPIO8: J4.10 (Pin_10), R7.2, U4.10 (GPIO8)
- new net GPIO9: J4.9 (Pin_9), R6.2, SW2.1, U4.15 (GPIO9)
- new net USB_DM: J2.A7 (D-), J2.B7 (D-), J4.12 (Pin_12), U3.3 (I/O2), U4.13 (GPIO12/USB_D-)
- new net USB_DP: J2.A6 (D+), J2.B6 (D+), J4.13 (Pin_13), U3.1 (I/O1), U4.14 (GPIO13/USB_D+)
- new net VBUS: C7.1, F2.1, U2.3 (VI), U3.6 (VBUS)
- no-connect marks 0 -> 5
Other:
- note added: "1) Rack only: +12V -> F1 -> D1 -> TPS54202 buck -> 3.43V (R1/R2 100k/21k, Vfb 0.596V) dominates +3V3"
- note added: "2) USB only (firmware): VBUS 5V -> F2 -> AMS1117-3.3 -> 3.3V"
- note added: "3) Both attached: buck (3.43V) sources the rail; AMS1117 idles (pass device off)"
- note added: "Antenna: keep copper-free under module antenna area (keepout zone included in footprint)."
- note added: "Doepfer 2x5: pins 1-2 = -12V (also J3 pin 3) | pins 3-8 = GND | pins 9-10 = +12V. Pin 1 = key side."
- note added: "Firmware: native ESP32-C6 USB-Serial/JTAG on IO12=D- / IO13=D+ (no CH340C needed)."
- note added: "J3/J4 expose all GPIOs + rails for carrier/breadboard. GPIO8/9 = strapping (10k PU) - do not hold low at reset. GPIO12/13 shared with USB."
- note added: "Power architecture:"
- note added: "RST (EN) + BOOT (IO9) buttons for manual download mode; USB-JTAG auto-resets into download."
- note added: "Strapping: IO9 10k PU (SPI boot) | IO8 10k PU | IO15 float (USB-JTAG default) | EN RC 10k + 1uF per datasheet."
- note added: "TPS54202 EN floated per TI datasheet (internal pull-up enables the converter)."
- company: (none) -> nanas sound
- title: (none) -> EuroPlatvorm - ESP32-C6 core + power

Commit message: Route EuroPlatvorm manually; fix GPIO labels and USB-C shell pad drills
Parts:
- J1: footprint Connector_IDC:IDC-Header_2x05_P2.54mm_Vertical -> Connector_PinHeader_2.54mm:PinHeader_2x05_P2.54mm_Vertical; LCSC C32713306 -> C492422; MPN PM2.54-2x5P-ZC -> PZ254V-12-10P
Connections:
- net GPIO10: now also J4.11 (Pin_11); no longer J3.12 (Pin_12)
- net GPIO11: now also J4.10 (Pin_10); no longer J4.11 (Pin_11)
- net GPIO15: now also J4.9 (Pin_9); no longer J3.13 (Pin_13)
- net GPIO16: now also J4.8 (Pin_8); no longer J4.7 (Pin_7)
- net GPIO17: now also J4.7 (Pin_7); no longer J4.8 (Pin_8)
- net GPIO18: now also J4.6 (Pin_6); no longer J4.1 (Pin_1)
- net GPIO19: now also J4.5 (Pin_5); no longer J4.2 (Pin_2)
- net GPIO20: now also J4.4 (Pin_4); no longer J4.3 (Pin_3)
- net GPIO21: now also J4.3 (Pin_3); no longer J4.4 (Pin_4)
- net GPIO22: now also J4.2 (Pin_2); no longer J4.5 (Pin_5)
- net GPIO23: now also J4.1 (Pin_1); no longer J4.6 (Pin_6)
- net GPIO8: now also J4.13 (Pin_13); no longer J4.10 (Pin_10)
- net GPIO9: now also J4.12 (Pin_12); no longer J4.9 (Pin_9)
- net USB_DM: now also J3.13 (Pin_13); no longer J4.12 (Pin_12)
- net USB_DP: now also J3.12 (Pin_12); no longer J4.13 (Pin_13)
Changed lines of the file:
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@@
 		)
 	)
-	(label "GPIO19"
+	(label "GPIO22"
 		(at 130.81 139.7 0)
 		(effects
@@
 		)
 	)
-	(label "GPIO22"
+	(label "GPIO19"
 		(at 130.81 147.32 0)
 		(effects
@@
 		)
 	)
-	(label "GPIO8"
+	(label "GPIO11"
 		(at 130.81 160.02 0)
 		(effects
@@
 		)
 	)
-	(label "GPIO16"
+	(label "GPIO17"
 		(at 130.81 152.4 0)
 		(effects
@@
 		)
 	)
-	(label "GPIO17"
+	(label "GPIO16"
 		(at 130.81 154.94 0)
 		(effects
@@
 		)
 	)
-	(label "GPIO23"
+	(label "GPIO18"
 		(at 130.81 149.86 0)
 		(effects
@@
 		)
 	)
-	(label "GPIO15"
+	(label "USB_DM"
 		(at 113.03 167.64 180)
 		(effects
@@
 		)
 	)
-	(label "GPIO21"
+	(label "GPIO20"
 		(at 130.81 144.78 0)
 		(effects
@@
 		)
 	)
-	(label "GPIO18"
+	(label "GPIO23"
 		(at 130.81 137.16 0)
 		(effects
@@
 		)
 	)
-	(label "GPIO20"
+	(label "GPIO21"
 		(at 130.81 142.24 0)
 		(effects
@@
 		)
 	)
-	(label "GPIO9"
+	(label "GPIO15"
 		(at 130.81 157.48 0)
 		(effects
@@
 		)
 	)
-	(label "GPIO10"
+	(label "USB_DP"
 		(at 113.03 165.1 180)
 		(effects
@@
 		)
 	)
-	(label "GPIO11"
+	(label "GPIO10"
 		(at 130.81 162.56 0)
 		(effects
@@
 		)
 	)
-	(label "USB_DP"
+	(label "GPIO8"
 		(at 130.81 167.64 0)
 		(effects
@@
 		)
 	)
-	(label "USB_DM"
+	(label "GPIO9"
 		(at 130.81 165.1 0)
 		(effects
@@
 			)
 		)
-		(property "Footprint" "Connector_IDC:IDC-Header_2x05_P2.54mm_Vertical"
+		(property "Footprint" "Connector_PinHeader_2.54mm:PinHeader_2x05_P2.54mm_Vertical"
 			(at 34.29 39.37 0)
 			(hide yes)
@@
 			)
 		)
-		(property "Datasheet" "~"
+		(property "Datasheet" "https://datasheet.lcsc.com/datasheet/pdf/50ec9710cee52ae98bff43fbb8887c5b.pdf?productCode=C492422"
 			(at 34.29 39.37 0)
 			(hide yes)
@@
 			)
 		)
-		(property "MPN" "PM2.54-2x5P-ZC"
+		(property "MPN" "PZ254V-12-10P"
 			(at 34.29 39.37 0)
 			(hide yes)
@@
 			)
 		)
-		(property "LCSC" "C32713306"
+		(property "LCSC" "C492422"
 			(at 34.29 39.37 0)
 			(hide yes)

Commit message: Fix EMI review findings: C11 decoupling at 3V3 pin, buck SW/FB hot loop, USB routing, Vout to 3.3V
Parts:
- C11: footprint Capacitor_SMD:C_0603_1608Metric -> Capacitor_SMD:C_0402_1005Metric; LCSC C14663 -> C307331; MPN CC0603KRX7R9BB104 -> CL05B104KB5NNNC
- R2: value 21k -> 22k; LCSC C49653293 -> C2907015; MPN GR0603F21KT5G00 -> FRC0603F2202TS
Changed lines of the file:
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@@
 			)
 		)
-		(property "Value" "21k"
+		(property "Value" "22k"
 			(at 139.192 65.786 0)
 			(show_name no)
@@
 			)
 		)
-		(property "MPN" "GR0603F21KT5G00"
+		(property "MPN" "FRC0603F2202TS"
 			(at 137.16 66.04 0)
 			(hide yes)
@@
 			)
 		)
-		(property "LCSC" "C49653293"
+		(property "LCSC" "C2907015"
 			(at 137.16 66.04 0)
 			(hide yes)
@@
 			)
 		)
-		(property "Footprint" "Capacitor_SMD:C_0603_1608Metric"
+		(property "Footprint" "Capacitor_SMD:C_0402_1005Metric"
 			(at 236.22 67.31 0)
 			(hide yes)
@@
 			)
 		)
-		(property "MPN" "CC0603KRX7R9BB104"
+		(property "MPN" "CL05B104KB5NNNC"
 			(at 236.22 67.31 0)
 			(hide yes)
@@
 			)
 		)
-		(property "LCSC" "C14663"
+		(property "LCSC" "C307331"
 			(at 236.22 67.31 0)
 			(hide yes)

Commit message: Fix USBLC6-2SC6 pin map blocker, re-route U3 area, refresh gerbers
- Symbol (platvorm.kicad_sym + embedded copy): pin4=I/O2, pin5=VBUS
  (power_in), pin6=I/O1 per ST datasheet Fig 1 (was NC/NC/VBUS)
- Schematic: VBUS label moved to pin 5 stub; USB_DM/USB_DP labels on
  pins 4/6; two no-connect flags removed
- PCB: pads 4/5/6 re-netted; USB_DP tie pads 6-1; USB_DM via-hop
  pad4 -> B.Cu -> via (135.5,127.5); VBUS jogged to pad 5 with F.Cu
  bridge through x=137.93 channel; F2-Pad2 escape wall rerouted to
  x=138.4 around J2 pad3/pad4
- 22uF value strings corrected to 6.3V (matches CL21A226MQQNNNE)
- B.Silkscreen sketch art scaled 0.984 + recentered to fit outline
  (was clipping 0.43mm past board edge)
- Zones refilled; kicad-cli DRC clean on clearance/tracks/unconnected;
  gerbers + drill + job re-exported; U3 pad nets verified in F_Cu.gbr
Parts:
- C10, C4, C5, C8: value 22uF 10V -> 22uF 6.3V
Connections:
- net USB_DM: now also U3.4 (I/O2)
- net USB_DP: now also U3.6 (I/O1)
- net VBUS: now also U3.5 (VBUS); no longer U3.6 (VBUS)
- no-connect marks 5 -> 3
Changed lines of the file:
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@@
 	)
 	(no_connect
-		(at 62.23 161.29)
-	)
-	(no_connect
-		(at 62.23 156.21)
-	)
-	(no_connect
 		(at 66.04 118.11)
 	)
@@
 		)
 	)
-	(label "VBUS"
+	(label "USB_DM"
+		(at 67.31 161.29 0)
+		(effects
+			(font
+				(size 1.27 1.27)
+			)
+			(justify left bottom)
+		)
+	)
+	(label "USB_DP"
 		(at 67.31 151.13 0)
 		(effects
@@
 		)
 	)
+	(label "VBUS"
+		(at 67.31 156.21 0)
+		(effects
+			(font
+				(size 1.27 1.27)
+			)
+			(justify left bottom)
+		)
+	)
+	(wire
+		(pts
+			(xy 62.23 156.21)
+			(xy 67.31 156.21)
+		)
+		(stroke
+			(width 0)
+			(type default)
+		)
+	)
+	(wire
+		(pts
+			(xy 62.23 161.29)
+			(xy 67.31 161.29)
+		)
+		(stroke
+			(width 0)
+			(type default)
+		)
+	)
 	(label "GPIO16"
 		(at 130.81 154.94 0)
@@
 			)
 		)
-		(property "Value" "22uF 10V"
+		(property "Value" "22uF 6.3V"
 			(at 162.052 43.18 0)
 			(show_name no)
@@
 			)
 		)
-		(property "Value" "22uF 10V"
+		(property "Value" "22uF 6.3V"
 			(at 150.114 43.18 0)
 			(show_name no)
@@
 			)
 		)
-		(property "Value" "22uF 10V"
+		(property "Value" "22uF 6.3V"
 			(at 137.922 106.68 0)
 			(show_name no)
@@
 			)
 		)
-		(property "Value" "22uF 10V"
+		(property "Value" "22uF 6.3V"
 			(at 233.172 69.85 0)
 			(show_name no)

Commit message: Fix C7 MPN/footprint mismatch: swap to 0805 CL21A106KPCLQNC (C962097)
Board footprint is 0805 but the BOM part CL10A106KP8NNNC (C19702) is
physically 0603, so fab would source a 0603 chip for 0805 pads. Swap
MPN/LCSC in schematic, PCB, and exported BOM; footprint unchanged.
Parts:
- C7: LCSC C19702 -> C962097; MPN CL10A106KP8NNNC -> CL21A106KPCLQNC
Changed lines of the file:
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@@
 			)
 		)
-		(property "MPN" "CL10A106KP8NNNC"
+		(property "MPN" "CL21A106KPCLQNC"
 			(at 96.52 104.14 0)
 			(hide yes)
@@
 			)
 		)
-		(property "LCSC" "C19702"
+		(property "LCSC" "C962097"
 			(at 96.52 104.14 0)
 			(hide yes)
